File: hardware/kicad/glitchwave567/glitchwave567.kicad_sch (KiCad schematic)
At the start: 0 parts

Commit message: hardware: root hierarchy + ERC pass on KiCad 10 (down to lib-mismatch/footprint noise + 2 intentional OTA current-sum waivers)
- root sheet ties all 8 sheets into one project (global-label connectivity, 288 comps / 259 nets stitch verified)
- fixed: U11/U12->U18/U19 ref clash, MCU cap ref clashes, env rectifier D81 feedback returned to virtual ground (was floating FW_IN2), PWR_FLAGs on PICO_VSYS + ctrl rails, off-grid buffer pin
- remaining ERC: footprint_link (assignment pending), lib_symbol_mismatch (v6 embedded vs v10 libs, cosmetic), 2x pin_to_pin Output-Output = LM13700 current summing (by design, noted on sheets)

Co-Authored-By: Claude Fable 5 <noreply@anthropic.com>
Other:
- added sheet core567 (core567.kicad_sch)
- added sheet env_cv (env_cv.kicad_sch)
- added sheet input_dirt (input_dirt.kicad_sch)
- added sheet jacks (jacks.kicad_sch)
- added sheet mcu (mcu.kicad_sch)
- added sheet mix_svf (mix_svf.kicad_sch)
- added sheet output (output.kicad_sch)
- added sheet power (power.kicad_sch)
- note added: "GLITCHWAVE 567 — digitally-controlled analog. All inter-sheet nets are GLOBAL LABELS; sheets below are containers."
- note added: "Signal: jacks -> input_dirt -> core567 -> mix_svf -> output -> jacks. Control: mcu PWM CVs everywhere. Power: power."
- title: Glitchwave 567 -> Glitchwave 567 — Main Board (root)
Changed lines of the file:
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@@
-(kicad_sch (version 20230121) (generator claude)
+(kicad_sch (version 20211014) (generator schgen)
   (paper "A3")
-  (title_block (title "Glitchwave 567") (company "Illicit Apothecary") (rev "0.1"))
+  (title_block
+    (title "Glitchwave 567 — Main Board (root)")
+    (rev "0.1")
+    (company "Illicit Apothecary")
+  )
+  (text "GLITCHWAVE 567 — digitally-controlled analog. All inter-sheet nets are GLOBAL LABELS; sheets below are containers."
+    (at 25.4 25.4 0)
+    (effects (font (size 2.2 2.2)))
+  )
+  (text "Signal: jacks -> input_dirt -> core567 -> mix_svf -> output -> jacks. Control: mcu PWM CVs everywhere. Power: power."
+    (at 25.4 30.48 0)
+    (effects (font (size 1.8 1.8)))
+  )
+  (sheet (at 33.02 45.72) (size 63.5 38.1)
+    (stroke (width 0.1524) (type solid))
+    (fill (color 0 0 0 0))
+    (property "Sheet name" "power" (at 33.02 44.92 0)
+      (effects (font (size 1.6 1.6)))
+    )
+    (property "Sheet file" "power.kicad_sch" (at 33.02 84.62 0)
+      (effects (font (size 1.27 1.27)))
+    )
+  )
+  (sheet (at 121.92000000000002 45.72) (size 63.5 38.1)
+    (stroke (width 0.1524) (type solid))
+    (fill (color 0 0 0 0))
+    (property "Sheet name" "input_dirt" (at 121.92000000000002 44.92 0)
+      (effects (font (size 1.6 1.6)))
+    )
+    (property "Sheet file" "input_dirt.kicad_sch" (at 121.92000000000002 84.62 0)
+      (effects (font (size 1.27 1.27)))
+    )
+  )
+  (sheet (at 210.82000000000002 45.72) (size 63.5 38.1)
+    (stroke (width 0.1524) (type solid))
+    (fill (color 0 0 0 0))
+    (property "Sheet name" "core567" (at 210.82000000000002 44.92 0)
+      (effects (font (size 1.6 1.6)))
+    )
+    (property "Sheet file" "core567.kicad_sch" (at 210.82000000000002 84.62 0)
+      (effects (font (size 1.27 1.27)))
+    )
+  )
+  (sheet (at 299.72 45.72) (size 63.5 38.1)
+    (stroke (width 0.1524) (type solid))
+    (fill (color 0 0 0 0))
+    (property "Sheet name" "mix_svf" (at 299.72 44.92 0)
+      (effects (font (size 1.6 1.6)))
+    )
+    (property "Sheet file" "mix_svf.kicad_sch" (at 299.72 84.62 0)
+      (effects (font (size 1.27 1.27)))
+    )
+  )
+  (sheet (at 33.02 109.22) (size 63.5 38.1)
+    (stroke (width 0.1524) (type solid))
+    (fill (color 0 0 0 0))
+    (property "Sheet name" "output" (at 33.02 108.42 0)
+      (effects (font (size 1.6 1.6)))
+    )
+    (property "Sheet file" "output.kicad_sch" (at 33.02 148.12 0)
+      (effects (font (size 1.27 1.27)))
+    )
+  )
+  (sheet (at 121.92000000000002 109.22) (size 63.5 38.1)
+    (stroke (width 0.1524) (type solid))
+    (fill (color 0 0 0 0))
+    (property "Sheet name" "env_cv" (at 121.92000000000002 108.42 0)
+      (effects (font (size 1.6 1.6)))
+    )
+    (property "Sheet file" "env_cv.kicad_sch" (at 121.92000000000002 148.12 0)
+      (effects (font (size 1.27 1.27)))
+    )
+  )
+  (sheet (at 210.82000000000002 109.22) (size 63.5 38.1)
+    (stroke (width 0.1524) (type solid))
+    (fill (color 0 0 0 0))
+    (property "Sheet name" "mcu" (at 210.82000000000002 108.42 0)
+      (effects (font (size 1.6 1.6)))
+    )
+    (property "Sheet file" "mcu.kicad_sch" (at 210.82000000000002 148.12 0)
+      (effects (font (size 1.27 1.27)))
+    )
+  )
+  (sheet (at 299.72 109.22) (size 63.5 38.1)
+    (stroke (width 0.1524) (type solid))
+    (fill (color 0 0 0 0))
+    (property "Sheet name" "jacks" (at 299.72 108.42 0)
+      (effects (font (size 1.6 1.6)))
+    )
+    (property "Sheet file" "jacks.kicad_sch" (at 299.72 148.12 0)
+      (effects (font (size 1.27 1.27)))
+    )
+  )
+  (sheet_instances
+    (path "/e801c1e6-17ce-4ac2-a5fb-ac59051baef3" (page "2"))
+    (path "/1a8319a9-a6c2-4fef-b2a8-8e073003154a" (page "3"))
+    (path "/1df45449-3d65-473b-9336-38c51203ac43" (page "4"))
+    (path "/3f9dec00-ae75-4986-b3a2-98f6d4e97a80" (page "5"))
+    (path "/76e580bd-7276-48f8-89e3-7a546b45efe9" (page "6"))
+    (path "/c5e87dd4-2360-44c5-93cb-746d024435a9" (page "7"))
+    (path "/42babe6a-7070-407a-b036-269c6f78cc00" (page "8"))
+    (path "/481cb742-4c6a-409b-85ea-72199d372a5c" (page "9"))
+  )
 )
