File: hardware/kicad/glitchwave567/core567.kicad_sch (KiCad schematic)
At the start: 32 parts, among them Q2 MMBT3904, Q3 MMBT3904, U5 LM567 (SO-8), U7 LM13700, U8 CD4052B

Commit message: hardware: datasheet review pass - 13 fixes incl. 2 fatal (MP1584 pin scramble, SVF feedback dividers)
HIGH: MP1584 symbol pins remapped to real SOIC-8; EN divider 24k9 added (18V
on a 6V-max pin); SVF integrator 220k/680 feedback dividers + 220p caps
(was tuning to 611kHz); LM13700 buffer 10k DC loads; 78L09->1N4148W drop
(LM567C 9V abs max); bell EQ redesigned (was electrically inert - now exact
+3.04dB@790Hz Q=0.500); Pico ADC_VREF external feed removed (onboard ref).
MED: FREQ_CV 2nd PWM pole (-112dB, pitch FM), env attack 3.9k (exact 4ms),
567 pin3 1k clamp limit, SMAJ18A on VA, 50V input cap, buffer parking.
Full report: hardware/SCHEMATIC_REVIEW.md. All sheets re-verified.

Co-Authored-By: Claude Fable 5 <noreply@anthropic.com>
Parts:
- added R53: 1k (pin3 clamp-current limit), symbol Device:R
Connections:
- net GND: now also U7.10, U7.7
- net IN567: now also R53.2; no longer C3.2
- new net IN567A: C3.2, R53.1
- no-connect marks 12 -> 10
Other:
- note added: "OTA-off f0 accuracy/drift unspecified (fine: floor only). Mux rON adds ~3.6*rON/Reff timing error - firmware cal per range."
- note added: "R38 100k floor keeps the VCO alive at Iabc=0. NOTE: 100k is outside the 2k-20k documented RT range -"
- note removed: "R38 100k parallel floor keeps the VCO alive at Iabc=0. Original was R6 3.6k + B10k pot with C4 220n (304-1148Hz)."
Changed lines of the file:
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@@
   (no_connect (at 78.74 190.5))
   (no_connect (at 63.5 190.5))
-  (no_connect (at 88.9 190.5))
   (no_connect (at 99.06 193.04))
-  (no_connect (at 106.68 190.5))
   (no_connect (at 116.84 193.04))
   (wire (pts (xy 64.77 52.07) (xy 62.23 52.07))
@@
     (stroke (width 0.0))
   )
-  (wire (pts (xy 36.83 55.88) (xy 34.29 55.88))
-    (stroke (width 0.0))
-  )
-  (wire (pts (xy 44.45 55.88) (xy 46.99 55.88))
+  (wire (pts (xy 26.67 55.88) (xy 24.13 55.88))
+    (stroke (width 0.0))
+  )
+  (wire (pts (xy 34.29 55.88) (xy 36.83 55.88))
+    (stroke (width 0.0))
+  )
+  (wire (pts (xy 44.45 55.88) (xy 41.91 55.88))
+    (stroke (width 0.0))
+  )
+  (wire (pts (xy 52.07 55.88) (xy 54.61 55.88))
     (stroke (width 0.0))
   )
@@
   )
   (wire (pts (xy 78.74 193.04) (xy 81.28 193.04))
+    (stroke (width 0.0))
+  )
+  (wire (pts (xy 88.9 190.5) (xy 86.36 190.5))
+    (stroke (width 0.0))
+  )
+  (wire (pts (xy 106.68 190.5) (xy 104.14 190.5))
     (stroke (width 0.0))
   )
@@
     (effects (font (size 1.8 1.8)))
   )
-  (text "R38 100k parallel floor keeps the VCO alive at Iabc=0. Original was R6 3.6k + B10k pot with C4 220n (304-1148Hz)."
+  (text "R38 100k floor keeps the VCO alive at Iabc=0. NOTE: 100k is outside the 2k-20k documented RT range -"
     (at 25.4 100.33 0)
+    (effects (font (size 1.8 1.8)))
+  )
+  (text "OTA-off f0 accuracy/drift unspecified (fine: floor only). Mux rON adds ~3.6*rON/Reff timing error - firmware cal per range."
+    (at 25.4 104.14 0)
     (effects (font (size 1.8 1.8)))
   )
@@
     (effects (font (size 1.27 1.27)))
   )
-  (label "IN567" (at 46.99 55.88 0)
+  (label "IN567A" (at 36.83 55.88 0)
+    (effects (font (size 1.27 1.27)))
+  )
+  (label "IN567A" (at 41.91 55.88 180)
+    (effects (font (size 1.27 1.27)))
+  )
+  (label "IN567" (at 54.61 55.88 0)
     (effects (font (size 1.27 1.27)))
   )
@@
     (effects (font (size 1.27 1.27)))
   )
-  (global_label "V567_DRIVE" (shape bidirectional) (at 34.29 55.88 180)
+  (global_label "V567_DRIVE" (shape bidirectional) (at 24.13 55.88 180)
     (effects (font (size 1.27 1.27)))
   )
@@
   )
   (global_label "GND" (shape bidirectional) (at 81.28 193.04 0)
+    (effects (font (size 1.27 1.27)))
+  )
+  (global_label "GND" (shape bidirectional) (at 86.36 190.5 180)
+    (effects (font (size 1.27 1.27)))
+  )
+  (global_label "GND" (shape bidirectional) (at 104.14 190.5 180)
     (effects (font (size 1.27 1.27)))
   )
@@
     )
   )
-  (symbol (lib_id "Device:C") (at 40.64 55.88 90) (unit 1)
+  (symbol (lib_id "Device:C") (at 30.48 55.88 90) (unit 1)
     (in_bom yes) (on_board yes) (dnp no)
-    (property "Reference" "C3" (id 0) (at 40.64 53.34 0)
+    (property "Reference" "C3" (id 0) (at 30.48 53.34 0)
       (effects (font (size 1.27 1.27)))
     )
-    (property "Value" "220n" (id 1) (at 40.64 58.42 0)
+    (property "Value" "220n" (id 1) (at 30.48 58.42 0)
       (effects (font (size 1.27 1.27)))
     )
-    (property "Footprint" "" (id 2) (at 40.64 55.88 0)
+    (property "Footprint" "" (id 2) (at 30.48 55.88 0)
       (effects (font (size 1.27 1.27)) hide)
     )
-    (property "Datasheet" "" (id 3) (at 40.64 55.88 0)
+    (property "Datasheet" "" (id 3) (at 30.48 55.88 0)
       (effects (font (size 1.27 1.27)) hide)
     )
@@
         )
       )
+    )
+  )
+  (symbol (lib_id "Device:R") (at 48.26 55.88 90) (unit 1)
+    (in_bom yes) (on_board yes) (dnp no)
+    (property "Reference" "R53" (id 0) (at 48.26 53.34 0)
+      (effects (font (size 1.27 1.27)))
+    )
+    (property "Value" "1k (pin3 clamp-current limit)" (id 1) (at 48.26 58.42 0)
+      (effects (font (size 1.27 1.27)))
+    )
+    (property "Footprint" "" (id 2) (at 48.26 55.88 0)
+      (effects (font (size 1.27 1.27)) hide)
+    )
+    (property "Datasheet" "" (id 3) (at 48.26 55.88 0)
+      (effects (font (size 1.27 1.27)) hide)
+    )
+    (instances
+      (project "glitchwave567"
+        (path "/"
+          (reference "R53") (unit 1)
+        )
+      )

Commit message: hardware: footprint phase complete - 297/297 parts footprinted, custom Glitchwave.pretty authored from factory drawings
- Glitchwave.pretty: PJ-603A (pads 7.6/15.1/22.5, slots per HY-WI-32), PJ-3410,
  DC-044A (polarity DMM-verify flagged), ALPS_RK09K1130 (2.5 pitch + 8.8 snap
  legs from ALPS drawing), SSWFS-S01 (slot pads absorb 5.5-6.5 pin-spacing
  ambiguity; NOTE: PC-pin variant thread is 15/32-32 - panel hole D12.2+keyway,
  not M12), RPi_Pico_SMD (official Fig.5 land pattern, row c-c 19.38)
- schgen auto-footprint map wired into add(); all sheets regenerated
- fp-lib-tables for both projects; trims -> Bourns 3224W; clamps -> 1N5819W

Co-Authored-By: Claude Fable 5 <noreply@anthropic.com>
Parts:
- C3, C40, C41, C42, C43, C44, C45, C46, C49, C50: footprint (none) -> Capacitor_SMD:C_0603_1608Metric
- C47: footprint (none) -> Capacitor_SMD:CP_Elec_5x5.4
- C48: footprint (none) -> Capacitor_SMD:CP_Elec_10x10.2
- Q2, Q3: footprint (none) -> Package_TO_SOT_SMD:SOT-23
- R16, R38, R40, R41, R42, R43, R44, R45, R46, R47, R48, R49, R50, R51, R52, R53: footprint (none) -> Resistor_SMD:R_0603_1608Metric
- U5: footprint (none) -> Package_SO:SOIC-8_3.9x4.9mm_P1.27mm
- U7, U8: footprint (none) -> Package_SO:SOIC-16_3.9x9.9mm_P1.27mm
Changed lines of the file:
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@@
       (effects (font (size 1.27 1.27)))
     )
-    (property "Footprint" "" (id 2) (at 78.74 55.88 0)
+    (property "Footprint" "Package_SO:SOIC-8_3.9x4.9mm_P1.27mm" (id 2) (at 78.74 55.88 0)
       (effects (font (size 1.27 1.27)) hide)
     )
@@
       (effects (font (size 1.27 1.27)))
     )
-    (property "Footprint" "" (id 2) (at 30.48 55.88 0)
+    (property "Footprint" "Capacitor_SMD:C_0603_1608Metric" (id 2) (at 30.48 55.88 0)
       (effects (font (size 1.27 1.27)) hide)
     )
@@
       (effects (font (size 1.27 1.27)))
     )
-    (property "Footprint" "" (id 2) (at 48.26 55.88 0)
+    (property "Footprint" "Resistor_SMD:R_0603_1608Metric" (id 2) (at 48.26 55.88 0)
       (effects (font (size 1.27 1.27)) hide)
     )
@@
       (effects (font (size 1.27 1.27)))
     )
-    (property "Footprint" "" (id 2) (at 96.52 30.48 0)
+    (property "Footprint" "Capacitor_SMD:C_0603_1608Metric" (id 2) (at 96.52 30.48 0)
       (effects (font (size 1.27 1.27)) hide)
     )
@@
       (effects (font (size 1.27 1.27)))
     )
-    (property "Footprint" "" (id 2) (at 120.65 55.88 0)
+    (property "Footprint" "Capacitor_SMD:C_0603_1608Metric" (id 2) (at 120.65 55.88 0)
       (effects (font (size 1.27 1.27)) hide)
     )
@@
       (effects (font (size 1.27 1.27)))
     )
-    (property "Footprint" "" (id 2) (at 133.35 55.88 0)
+    (property "Footprint" "Capacitor_SMD:C_0603_1608Metric" (id 2) (at 133.35 55.88 0)
       (effects (font (size 1.27 1.27)) hide)
     )
@@
       (effects (font (size 1.27 1.27)))
     )
-    (property "Footprint" "" (id 2) (at 168.91 45.72 0)
+    (property "Footprint" "Resistor_SMD:R_0603_1608Metric" (id 2) (at 168.91 45.72 0)
       (effects (font (size 1.27 1.27)) hide)
     )
@@
       (effects (font (size 1.27 1.27)))
     )
-    (property "Footprint" "" (id 2) (at 181.61 63.5 0)
+    (property "Footprint" "Capacitor_SMD:C_0603_1608Metric" (id 2) (at 181.61 63.5 0)
       (effects (font (size 1.27 1.27)) hide)
     )
@@
       (effects (font (size 1.27 1.27)))
     )
-    (property "Footprint" "" (id 2) (at 196.85 45.72 0)
+    (property "Footprint" "Resistor_SMD:R_0603_1608Metric" (id 2) (at 196.85 45.72 0)
       (effects (font (size 1.27 1.27)) hide)
     )
@@
       (effects (font (size 1.27 1.27)))
     )
-    (property "Footprint" "" (id 2) (at 214.63 45.72 0)
+    (property "Footprint" "Resistor_SMD:R_0603_1608Metric" (id 2) (at 214.63 45.72 0)
       (effects (font (size 1.27 1.27)) hide)
     )
@@
       (effects (font (size 1.27 1.27)))
     )
-    (property "Footprint" "" (id 2) (at 214.63 63.5 0)
+    (property "Footprint" "Resistor_SMD:R_0603_1608Metric" (id 2) (at 214.63 63.5 0)
       (effects (font (size 1.27 1.27)) hide)
     )
@@
       (effects (font (size 1.27 1.27)))
     )
-    (property "Footprint" "" (id 2) (at 33.02 116.84 0)
+    (property "Footprint" "Resistor_SMD:R_0603_1608Metric" (id 2) (at 33.02 116.84 0)
       (effects (font (size 1.27 1.27)) hide)
     )
@@
       (effects (font (size 1.27 1.27)))
     )
-    (property "Footprint" "" (id 2) (at 33.02 134.62 0)
+    (property "Footprint" "Resistor_SMD:R_0603_1608Metric" (id 2) (at 33.02 134.62 0)
       (effects (font (size 1.27 1.27)) hide)
     )
@@
       (effects (font (size 1.27 1.27)))
     )
-    (property "Footprint" "" (id 2) (at 45.72 134.62 0)
+    (property "Footprint" "Capacitor_SMD:C_0603_1608Metric" (id 2) (at 45.72 134.62 0)
       (effects (font (size 1.27 1.27)) hide)
     )
@@
       (effects (font (size 1.27 1.27)))
     )
-    (property "Footprint" "" (id 2) (at 58.42 116.84 0)
+    (property "Footprint" "Resistor_SMD:R_0603_1608Metric" (id 2) (at 58.42 116.84 0)
       (effects (font (size 1.27 1.27)) hide)
     )
@@
       (effects (font (size 1.27 1.27)))
     )
-    (property "Footprint" "" (id 2) (at 71.12 134.62 0)
+    (property "Footprint" "Resistor_SMD:R_0603_1608Metric" (id 2) (at 71.12 134.62 0)
       (effects (font (size 1.27 1.27)) hide)
     )
@@
       (effects (font (size 1.27 1.27)))
     )
-    (property "Footprint" "" (id 2) (at 83.82 134.62 0)
+    (property "Footprint" "Resistor_SMD:R_0603_1608Metric" (id 2) (at 83.82 134.62 0)
       (effects (font (size 1.27 1.27)) hide)
     )
@@
       (effects (font (size 1.27 1.27)))
     )
-    (property "Footprint" "" (id 2) (at 106.68 116.84 0)
+    (property "Footprint" "Package_SO:SOIC-16_3.9x9.9mm_P1.27mm" (id 2) (at 106.68 116.84 0)
       (effects (font (size 1.27 1.27)) hide)
     )
@@
       (effects (font (size 1.27 1.27)))
     )
-    (property "Footprint" "" (id 2) (at 83.82 152.4 0)
+    (property "Footprint" "Resistor_SMD:R_0603_1608Metric" (id 2) (at 83.82 152.4 0)
       (effects (font (size 1.27 1.27)) hide)
     )
@@
       (effects (font (size 1.27 1.27)))
     )
-    (property "Footprint" "" (id 2) (at 129.54 116.84 0)
+    (property "Footprint" "Resistor_SMD:R_0603_1608Metric" (id 2) (at 129.54 116.84 0)
       (effects (font (size 1.27 1.27)) hide)
     )
@@
       (effects (font (size 1.27 1.27)))
     )
-    (property "Footprint" "" (id 2) (at 190.5 127.0 0)
+    (property "Footprint" "Package_SO:SOIC-16_3.9x9.9mm_P1.27mm" (id 2) (at 190.5 127.0 0)
       (effects (font (size 1.27 1.27)) hide)
     )
@@
       (effects (font (size 1.27 1.27)))
     )
-    (property "Footprint" "" (id 2) (at 220.98 146.05 0)
+    (property "Footprint" "Capacitor_SMD:C_0603_1608Metric" (id 2) (at 220.98 146.05 0)
       (effects (font (size 1.27 1.27)) hide)
     )
@@
       (effects (font (size 1.27 1.27)))
     )
-    (property "Footprint" "" (id 2) (at 233.68 146.05 0)
+    (property "Footprint" "Capacitor_SMD:C_0603_1608Metric" (id 2) (at 233.68 146.05 0)
       (effects (font (size 1.27 1.27)) hide)
     )
@@
       (effects (font (size 1.27 1.27)))
     )
-    (property "Footprint" "" (id 2) (at 246.38 146.05 0)
+    (property "Footprint" "Capacitor_SMD:CP_Elec_5x5.4" (id 2) (at 246.38 146.05 0)
       (effects (font (size 1.27 1.27)) hide)
     )
@@
       (effects (font (size 1.27 1.27)))
     )
-    (property "Footprint" "" (id 2) (at 259.08 146.05 0)
+    (property "Footprint" "Capacitor_SMD:CP_Elec_10x10.2" (id 2) (at 259.08 146.05 0)
       (effects (font (size 1.27 1.27)) hide)
     )
@@
       (effects (font (size 1.27 1.27)))
     )
-    (property "Footprint" "" (id 2) (at 220.98 109.22 0)
+    (property "Footprint" "Capacitor_SMD:C_0603_1608Metric" (id 2) (at 220.98 109.22 0)
       (effects (font (size 1.27 1.27)) hide)
     )
@@
       (effects (font (size 1.27 1.27)))
     )
-    (property "Footprint" "" (id 2) (at 259.08 190.5 0)
+    (property "Footprint" "Resistor_SMD:R_0603_1608Metric" (id 2) (at 259.08 190.5 0)
       (effects (font (size 1.27 1.27)) hide)
     )
@@
       (effects (font (size 1.27 1.27)))
     )
-    (property "Footprint" "" (id 2) (at 269.24 190.5 0)
+    (property "Footprint" "Package_TO_SOT_SMD:SOT-23" (id 2) (at 269.24 190.5 0)
       (effects (font (size 1.27 1.27)) hide)
     )
@@
       (effects (font (size 1.27 1.27)))
     )
-    (property "Footprint" "" (id 2) (at 269.24 170.18 0)
+    (property "Footprint" "Resistor_SMD:R_0603_1608Metric" (id 2) (at 269.24 170.18 0)
       (effects (font (size 1.27 1.27)) hide)
     )
@@
       (effects (font (size 1.27 1.27)))
     )
-    (property "Footprint" "" (id 2) (at 280.66999999999996 190.5 0)
+    (property "Footprint" "Resistor_SMD:R_0603_1608Metric" (id 2) (at 280.66999999999996 190.5 0)
       (effects (font (size 1.27 1.27)) hide)
     )
@@
       (effects (font (size 1.27 1.27)))
     )
-    (property "Footprint" "" (id 2) (at 290.83 190.5 0)
+    (property "Footprint" "Package_TO_SOT_SMD:SOT-23" (id 2) (at 290.83 190.5 0)
       (effects (font (size 1.27 1.27)) hide)
     )
@@
       (effects (font (size 1.27 1.27)))
     )
-    (property "Footprint" "" (id 2) (at 290.83 170.18 0)
+    (property "Footprint" "Resistor_SMD:R_0603_1608Metric" (id 2) (at 290.83 170.18 0)
       (effects (font (size 1.27 1.27)) hide)
     )
@@
       (effects (font (size 1.27 1.27)))
     )
-    (property "Footprint" "" (id 2) (at 33.02 190.5 0)
+    (property "Footprint" "Package_SO:SOIC-16_3.9x9.9mm_P1.27mm" (id 2) (at 33.02 190.5 0)
       (effects (font (size 1.27 1.27)) hide)
     )
@@
       (effects (font (size 1.27 1.27)))
     )
-    (property "Footprint" "" (id 2) (at 48.26 190.5 0)
+    (property "Footprint" "Capacitor_SMD:C_0603_1608Metric" (id 2) (at 48.26 190.5 0)
       (effects (font (size 1.27 1.27)) hide)
     )
@@
       (effects (font (size 1.27 1.27)))
     )
-    (property "Footprint" "" (id 2) (at 71.12 190.5 0)
+    (property "Footprint" "Package_SO:SOIC-16_3.9x9.9mm_P1.27mm" (id 2) (at 71.12 190.5 0)
       (effects (font (size 1.27 1.27)) hide)
     )
@@
       (effects (font (size 1.27 1.27)))
     )
-    (property "Footprint" "" (id 2) (at 96.52 190.5 0)
+    (property "Footprint" "Package_SO:SOIC-16_3.9x9.9mm_P1.27mm" (id 2) (at 96.52 190.5 0)
       (effects (font (size 1.27 1.27)) hide)
     )
@@
       (effects (font (size 1.27 1.27)))
     )
-    (property "Footprint" "" (id 2) (at 114.3 190.5 0)
-      (effects (font (size 1.27 1.27)) hide)
-    )
+    (property "Footprint" "Package_SO:SOIC-16_3.9x9.9mm_P1.27mm" (id 2) (at 114.3 190.5 0)
+      (effects (font (size 1.27 1.27)) hide)
+    )

Commit message: hardware: fix C107 duplicate refdes, add missing courtyards, rename silkscreen
Pre-order verification pass before sending the boards to PCBWay. Full write-up in
hardware/fab/ORDER_READINESS_20260911.md.

C107 was a duplicate reference designator: a 100n 0603 on FREQ_CV in mcu.kicad_sch
and a 22uF 0805 in power.kicad_sch that is the MP1584's second output capacitor.
Only the 100n existed on the PCB, so the +5V rail (Pico plus six WS2812B via J10)
would have been built with half its intended bulk capacitance, and the BOM listed
C107 twice with conflicting parts. KiCad collapses a duplicate refdes to one
component, so footprint count matched symbol count, DRC schematic parity passed and
ERC said nothing. Only a designator-level BOM-vs-board-vs-CPL diff finds it.

  - power.kicad_sch: the 22uF symbol renamed C107 to C112
  - MAIN PCB: C112 placed at (62.6, 25.0), 0.3mm F.Cu stub to the +5V trunk at
    y=23.65, GND through the F.Cu pour exactly as C108 is connected. Placement
    chosen by a clearance search, nearest obstacle 0.42mm against a 0.13mm rule.
    No via: every via position in that pocket scored under 0.23mm against the
    In2.Cu diagonals. Zones refilled.
  - BOM.xlsx: the 22uF row's designators changed from C107,C108 to C108,C112

Courtyards added to the 13 footprints that had none (J1-J6 and U20 on MAIN,
RV1-RV6 on CONTROL), copied from the library footprints. DRC was structurally blind
to body collisions on exactly the largest mechanical parts, which is why both jack
collisions went undetected in July. Every footprint on both boards now has one.
That exposed two more courtyard overlaps on MAIN, both courtyard-only with the
bodies clear: J5 to FB100 (0.700mm of body air, ~0.21mm of copper) and J4 to R98
(0.338mm). Nothing was moved because nothing collides.

Silkscreen on both boards renamed from "GLITCHWAVE 567" to "WHERE THE FUZZ MEETS
THE FUNK". Font 1.2 to 1.0mm so the longer string keeps about the same width:
measured in the plotted gerber it spans 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
Parts:
- C48: footprint Capacitor_SMD:CP_Elec_10x10.2 -> Capacitor_SMD:CP_Elec_10x10
Changed lines of the file:
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@@
       (effects (font (size 1.27 1.27)))
     )
-    (property "Footprint" "Capacitor_SMD:CP_Elec_10x10.2" (id 2) (at 259.08 146.05 0)
+    (property "Footprint" "Capacitor_SMD:CP_Elec_10x10" (id 2) (at 259.08 146.05 0)
       (effects (font (size 1.27 1.27)) hide)
     )
