File: hardware/kicad/glitchwave567/glitchwave567.kicad_pcb (KiCad board)
At the start: 4 copper layers, 138 x 114 mm, 296 parts, among them J1 IN 6.35mm PJ-603A, J10 CTRL 2x8, J2 OUT 6.35mm PJ-603A, J3 CV1 IN 3.5mm PJ-3410, J4 CV2 IN 3.5mm PJ-3410, J5 DC_2.1mm, J6 CV OUT 3.5mm PJ-3410, Q1 MMBTA13, Q10 AO3401A, Q11 BCP56, Q2 MMBT3904, Q3 MMBT3904, Q4 MMBT3904, Q5 MMBT3904, Q6 MMBT3904, SW1 +6dB (short=OFF), SW2 JFET in/out, SW3 ladder in/out, U1 TL074, U10 LM13700, U11 LM13700, U12 LM13700, U13 CD4051B, U14 TL074, U15 LM13700, U16 TL074, U17 TL074, U18 L78L09, U19 MP1584EN, U2 TL074, U20 Raspberry Pi Pico, U21 74HC4067, U22 74AHCT1G125, U3 LM13700, U5 LM567 (SO-8), U6 TL074, U7 LM13700, U8 CD4052B, U9 TL074

Commit message: hardware: fix C107 duplicate refdes, add missing courtyards, rename silkscreen
Pre-order verification pass before sending the boards to PCBWay. Full write-up in
hardware/fab/ORDER_READINESS_20260911.md.

C107 was a duplicate reference designator: a 100n 0603 on FREQ_CV in mcu.kicad_sch
and a 22uF 0805 in power.kicad_sch that is the MP1584's second output capacitor.
Only the 100n existed on the PCB, so the +5V rail (Pico plus six WS2812B via J10)
would have been built with half its intended bulk capacitance, and the BOM listed
C107 twice with conflicting parts. KiCad collapses a duplicate refdes to one
component, so footprint count matched symbol count, DRC schematic parity passed and
ERC said nothing. Only a designator-level BOM-vs-board-vs-CPL diff finds it.

  - power.kicad_sch: the 22uF symbol renamed C107 to C112
  - MAIN PCB: C112 placed at (62.6, 25.0), 0.3mm F.Cu stub to the +5V trunk at
    y=23.65, GND through the F.Cu pour exactly as C108 is connected. Placement
    chosen by a clearance search, nearest obstacle 0.42mm against a 0.13mm rule.
    No via: every via position in that pocket scored under 0.23mm against the
    In2.Cu diagonals. Zones refilled.
  - BOM.xlsx: the 22uF row's designators changed from C107,C108 to C108,C112

Courtyards added to the 13 footprints that had none (J1-J6 and U20 on MAIN,
RV1-RV6 on CONTROL), copied from the library footprints. DRC was structurally blind
to body collisions on exactly the largest mechanical parts, which is why both jack
collisions went undetected in July. Every footprint on both boards now has one.
That exposed two more courtyard overlaps on MAIN, both courtyard-only with the
bodies clear: J5 to FB100 (0.700mm of body air, ~0.21mm of copper) and J4 to R98
(0.338mm). Nothing was moved because nothing collides.

Silkscreen on both boards renamed from "GLITCHWAVE 567" to "WHERE THE FUZZ MEETS
THE FUNK". Font 1.2 to 1.0mm so the longer string keeps about the same width:
measured in the plotted gerber it spans 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
Parts:
- added C112: 22u, C_0805_2012Metric, F.Cu at (62.6, 25.0)
Routing:
- net +5V: track 191.9 -> 193.3 mm
Other:
- board text added: "WHERE THE FUZZ MEETS THE FUNK - MAIN rev0.1 Illicit Apothecary"
- board text removed: "GLITCHWAVE 567 - MAIN rev0.1 Illicit Apothecary"

Commit message: Rev 8: third stomp (SW3) + STOMP3 to GP22, boards/BOM/fab package updated
CONTROL: SW3 at (69,96); SW1/SW2 outboard to 23.28/114.72 (1.800in pitch);
LED4/LED5 follow; C7 +1.5mm east; 3 GND stitch vias cleared from new pad rows;
/POT3_W detoured around SW2's new COM pad; stomp silk now A/B/C; STOMP3 on
spare J1 pin 15. Fixes schematic pin1/pin3 inversion on SW1/SW2 (GND belongs
on N.O.; PCB was already right). DRC 0 errors.

MAIN: R175 10k pullup + C125 100n added; STOMP3 routed J10.15 -> GP22 (Pico
pad 29). DRC/ERC at pre-existing baselines. BOM.xlsx updated (SW qty 3, R/C
qty bumps, stale Suntsu README lines replaced). Fab package regenerated both
boards: Glitchwave567_PCBWay_Release_20260921.zip, README_PCBWAY rev 0.6.

Enclosure drill template still stale: needs three D12.2 at centreline +/-45.72mm.

Co-Authored-By: Claude Fable 5 <noreply@anthropic.com>
Claude-Session: https://claude.ai/code/session_01ArRoxLtCyE7DZoHE3DcYLs
Parts:
- added C125: 100n, C_0603_1608Metric, F.Cu at (39.5, 112.6)
- added R175: 10k, R_0603_1608Metric, F.Cu at (112.0, 107.3)
Connections:
- J10 pad 15: unconnected-(J10-Pin_15-Pad15) -> /mcu/STOMP3
- U20 pad 29: unconnected-(U20-GP22-Pad29) -> /mcu/STOMP3
Routing:
- net /mcu/STOMP3: track 0.00 -> 118.3 mm, vias 0 -> 3
- net 3V3: track 298.0 -> 300.7 mm
- net GND: track 1.00 -> 2.36 mm, vias 128 -> 129
