File: hardware/kicad/glitchwave567_ctrl/glitchwave567_ctrl.kicad_pcb (KiCad board)
At the start: 4 copper layers, 138 x 114 mm, 22 parts, among them J1 to MAIN 2x8 (B.Cu, mirrored), SW1 Suntsu SSWFS-S01 (TAP/BYP), SW2 Suntsu SSWFS-S01 (TAP/BYP)

Commit message: hardware: clear every pre-order blocker - M3 standoff holes, complete BOM, connector pair chosen
Three blockers stood between this project and a turnkey order. All three are
closed. Both boards are now genuinely orderable.

1. CONTROL BOARD HAD NO MOUNTING HOLES AT ALL.
ENCLOSURE_FIT.md says "control-board retention must come from standoffs" and
lists four M3 holes in its own "Required changes before ordering" section.
They were never added - and the pots are snap-in with no nuts, so nothing
held that board in the enclosure. Ordering as-was would have produced five
unmountable control boards.

Added four Ø3.2 mm NPTH holes at (17, 9.5), (121, 9.5), (17, 108.5) and
(121, 108.5). Every position verified against the REAL Edge.Cuts outline -
this board has 11 x 11 mm corner notches, so a bounding-box test happily
proposes holes in thin air, which the first pass did. Clearances: >= 3.69 mm
to the nearest copper (a GND via in each case) and >= 5.5 mm to the board
edge. Symmetric about x = 69; the obvious y-symmetric positions at 104.5 and
5.5 both collide with GND vias, so the pattern is offset in y by design.
MAIN board deliberately gets none - six jack bushings with nuts through the
walls retain it. Confirmed in the regenerated NPTH drill file.

2. THE BOM WAS FAR LESS COMPLETE THAN THE FAB README CLAIMED.
The README said "every BOM line carries an LCSC C-number". It did not - 63 of
96 MAIN lines and 3 of 11 CONTROL lines had supplier part number "generic":
every resistor, every capacitor, the ferrite and both connectors. Mostly
survivable, but not for C104, whose whole point is 50 V X7R because of DC-bias
derating at 18 V, nor for the electrolytics whose case size must match the
footprint, nor for a 3 A ferrite.

All 64 lines backfilled with real, stock-checked LCSC parts. Selection rules:
JLC basic/preferred where it exists; 0603 1% for resistors; X7R/X5R/C0G only
for MLCC (Y5V and Z5U rejected outright); >= 25 V on the 9-18 V rail;
electrolytic case size matched EXAC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
Parts:
- added H1: M3 standoff, MountingHole_3.2mm_M3, F.Cu at (17.0, 9.50)
- added H2: M3 standoff, MountingHole_3.2mm_M3, F.Cu at (121.0, 9.50)
- added H3: M3 standoff, MountingHole_3.2mm_M3, F.Cu at (17.0, 108.5)
- added H4: M3 standoff, MountingHole_3.2mm_M3, F.Cu at (121.0, 108.5)
